File: Tuer.kicad_pcb (KiCad board)
At the start: 2 copper layers, 25 parts, among them CON1 Sound Out, CON2 Speach In, P1 Rasp17_36, P2 Blau, P3 Braun, P4 Weis, P5 Rot, P6 Orange, Q1 BD433, Q2 Q_PMOS_SGD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

Commit message: hopfully fixed missing libs
Parts:
- 4N2x1, 4N32, 4N32_2, 4N32_3: footprint Opto-Devices:Optocoupler_6pin_wide_Stile-II -> Housings_DIP:DIP-6_W7.62mm
- C1, C2: footprint Capacitors_ThroughHole:C_Rect_L7_W2_P5 -> Capacitors_ThroughHole:C_Radial_D5_L6_P2.5
- Q1: footprint Transistors_OldSowjetAera:OldSowjetaera_Transistor_Type-I_SmallPads -> Pin_Headers:Pin_Header_Straight_1x03
- Q2, Q3: value Q_PMOS_SGD -> Q_PMOS_GDS; footprint Transistors_OldSowjetAera:OldSowjetaera_Transistor_Type-I_SmallPads -> Pin_Headers:Pin_Header_Straight_1x03
- R1, R3: footprint Resistors_ThroughHole:Resistor_Ceramic_Horizontal_L23mm-W9mm-H9mm-p30mm -> Resistors_ThroughHole:Resistor_Horizontal_RM15mm
- R2: footprint Resistors_ThroughHole:Resistor_Ceramic_Horizontal_L23mm-W9mm-H9mm-p30mm -> Resistors_ThroughHole:Resistor_Horizontal_RM10mm
- R4, R5: footprint Resistors_ThroughHole:Resistor_Ceramic_Horizontal_L23mm-W9mm-H9mm-p30mm -> Resistors_ThroughHole:Resistor_Vertical_RM5mm
- moved CON2 98.0 mm to (66.0, 45.7), turned to 0 degrees
- moved C1 78.9 mm to (66.0, 58.4), turned to 90 degrees
- moved R1 59.3 mm to (104.1, 109.2), turned to 0 degrees
- moved R5 57.1 mm to (96.5, 66.0), turned to 270 degrees
- moved P5 55.7 mm to (102.9, 68.6)
- moved P4 54.4 mm to (105.4, 71.1)
- moved R2 53.9 mm to (73.7, 66.0)
- moved CON1 52.1 mm to (116.8, 66.0)
- moved Q2 51.2 mm to (78.7, 76.2), turned to 180 degrees
- moved 4N32_2 45.7 mm to (61.0, 61.0), turned to 0 degrees
- moved Q3 39.5 mm to (99.1, 63.5), turned to 0 degrees
- moved R4 34.2 mm to (73.7, 73.7), turned to 270 degrees
- moved SW1 29.7 mm to (71.1, 137.2)
- moved Q1 20.5 mm to (91.4, 119.4), turned to 180 degrees
- moved SP1 18.0 mm to (121.9, 86.4)
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Connections:
- Q2 pad 1: /12V -> Net-(4N32_3-Pad5)
- Q2 pad 2: Net-(4N32_3-Pad5) -> Net-(C1-Pad2)
- Q2 pad 3: Net-(C1-Pad2) -> /12V
- Q3 pad 1: /11V -> Net-(4N32_2-Pad5)
- Q3 pad 2: Net-(4N32_2-Pad5) -> Net-(CON1-Pad2)
- Q3 pad 3: Net-(CON1-Pad2) -> /11V
Routing:
- net Net-(4N2x1-Pad1): track 78.8 -> 5.08 mm, vias 1 -> 0
- net GND: track 157.2 -> 107.4 mm
- net Net-(4N32_3-Pad5): track 96.3 -> 51.9 mm
- net /11V: track 39.9 -> 6.37 mm, vias 1 -> 0
- net /12V: track 59.7 -> 31.8 mm
- net Earth: track 243.1 -> 216.3 mm
- net Net-(4N32-Pad4): track 40.9 -> 17.8 mm, vias 2 -> 0
- net Net-(C2-Pad1): track 7.62 -> 30.5 mm, vias 0 -> 1
- net Net-(C1-Pad2): track 26.9 -> 45.8 mm, vias 0 -> 2
- net Net-(CON1-Pad2): track 34.1 -> 17.9 mm
- net ActivateMic: track 89.1 -> 74.0 mm, vias 1 -> 2
- net Net-(C2-Pad2): track 25.4 -> 12.8 mm
- net /23,5V: track 60.4 -> 48.3 mm
- net Net-(Q1-Pad1): track 92.7 -> 80.7 mm, vias 1 -> 2
- net Net-(C1-Pad1): track 21.9 -> 32.5 mm, vias 0 -> 1
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