File: Tuer.sch (KiCad schematic (older format))
At the start: 25 parts, among them CON1 Sound Out, CON2 Speach In, P1 Rasp17_36, P2 Blau, P3 Braun, P4 Weis, P5 Rot, P6 Orange, Q1 BD433, Q2 Q_PMOS_SGD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

Commit message: hopfully fixed missing libs
Parts:
- removed Q2, Q3: Q_PMOS_SGD, Transistors_OldSowjetAera:OldSowjetaera_Transistor_Type-I_SmallPads, symbol Q_PMOS_SGD
- added Q2, Q3: Q_PMOS_GDS, Pin_Headers:Pin_Header_Straight_1x03, symbol Tuer-rescue:Q_PMOS_GDS
- 4N2x1, 4N32, 4N32_2, 4N32_3: footprint Opto-Devices:Optocoupler_6pin_wide_Stile-II -> Housings_DIP:DIP-6_W7.62mm; symbol OPTO-TRANSISTOR -> Tuer-rescue:OPTO-TRANSISTOR
- C1, C2: footprint Capacitors_ThroughHole:C_Rect_L7_W2_P5 -> Capacitors_ThroughHole:C_Radial_D5_L6_P2.5; symbol C -> Tuer-rescue:C
- CON1, CON2: symbol BARREL_JACK -> Tuer-rescue:BARREL_JACK
- KB817: symbol PC817 -> Tuer-rescue:PC817
- P1: symbol CONN_02X10 -> Tuer-rescue:CONN_02X10
- P2, P3, P4, P5, P6: symbol CONN_01X01 -> Tuer-rescue:CONN_01X01
- Q1: footprint Transistors_OldSowjetAera:OldSowjetaera_Transistor_Type-I_SmallPads -> Pin_Headers:Pin_Header_Straight_1x03; symbol BD433 -> Tuer-rescue:BD433
- R1, R3: footprint Resistors_ThroughHole:Resistor_Ceramic_Horizontal_L23mm-W9mm-H9mm-p30mm -> Resistors_ThroughHole:Resistor_Horizontal_RM15mm; symbol R -> Tuer-rescue:R
- R2: footprint Resistors_ThroughHole:Resistor_Ceramic_Horizontal_L23mm-W9mm-H9mm-p30mm -> Resistors_ThroughHole:Resistor_Horizontal_RM10mm; symbol R -> Tuer-rescue:R
- R4, R5: footprint Resistors_ThroughHole:Resistor_Ceramic_Horizontal_L23mm-W9mm-H9mm-p30mm -> Resistors_ThroughHole:Resistor_Vertical_RM5mm; symbol R -> Tuer-rescue:R
- SP1: symbol SPEAKER -> Tuer-rescue:SPEAKER
- SW1: symbol SW_PUSH -> Tuer-rescue:SW_PUSH
Connections:
- wire segments 65 -> 75
